File: DashSight-Mezzanine-Card.kicad_pcb (KiCad board)
At the start: 2 copper layers, 75.1 x 78.5 mm, 70 parts, among them IC1 XM1110, IC2 ELM327, J1 Pi2 Connector, J2 Euler Connector, J3 Conn_Coaxial, J4 OBD2-DB9_Male, Q1 2N3904, Q2 2N3906, Q3 2N3906, Q4 2N3904, Q5 2N3904, Q6 2N3904, Q7 2N3904, U1 MCP2561-E/P, U2 LM317L_TO92, U3 LM1085-5.0, U4 ADuM1201AR, Y1 4.0MHz

Commit message: Update with the official KiCAD XM1110
Signed-off-by: Alistair Francis <alistair@alistair23.me>
Parts:
- IC1: footprint DashSight-PCB-Footprints:Sierra_XM11X0 -> RF_GPS:Sierra_XM11X0
Changed lines of the file:
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@@
     (add_net "Net-(IC1-Pad2)")
+  )
+  (module RF_GPS:Sierra_XM11X0 (layer F.Cu)
+    (at 138.303 63.119 270)
+    (descr "QFN-20, Pitch 1.20 no EP, https://source.sierrawireless.com/resources/airprime/hardware_specs_user_guides/airprime_xm1100_product_technical_specification")
+    (tags "QFN-20 P1.20")
+    (attr smd)
+    (fp_text reference IC1 (at -3.1 -6.55 90) (layer F.SilkS)
+      (effects (font (size 1 1) (thickness 0.15)))
+    )
+    (fp_text value XM1110 (at 0 6.45 90) (layer F.Fab)
+      (effects (font (size 1 1) (thickness 0.15)))
+    )
+    (fp_line (start -4.6 -4.62) (end -3.6 -4.62) (layer F.SilkS) (width 0.12))
+    (fp_line (start 4.87 4.62) (end 4.87 3.62) (layer F.SilkS) (width 0.12))
+    (fp_line (start 3.87 4.62) (end 4.87 4.62) (layer F.SilkS) (width 0.12))
+    (fp_line (start -4.87 4.62) (end -4.87 3.62) (layer F.SilkS) (width 0.12))
+    (fp_line (start -3.87 4.62) (end -4.87 4.62) (layer F.SilkS) (width 0.12))
+    (fp_line (start 4.87 -4.62) (end 4.87 -3.62) (layer F.SilkS) (width 0.12))
+    (fp_line (start 3.87 -4.62) (end 4.87 -4.62) (layer F.SilkS) (width 0.12))
+    (fp_line (start 5.8 -5.8) (end -5.8 -5.8) (layer F.CrtYd) (width 0.05))
+    (fp_line (start 5.8 5.8) (end 5.8 -5.8) (layer F.CrtYd) (width 0.05))
+    (fp_line (start -5.8 5.8) (end 5.8 5.8) (layer F.CrtYd) (width 0.05))
+    (fp_line (start -5.8 -5.8) (end -5.8 5.8) (layer F.CrtYd) (width 0.05))
+    (fp_line (start 4.75 -4.5) (end 4.75 4.5) (layer F.Fab) (width 0.1))
+    (fp_line (start -3.75 -4.5) (end 4.75 -4.5) (layer F.Fab) (width 0.1))
+    (fp_line (start -4.75 -3.5) (end -3.75 -4.5) (layer F.Fab) (width 0.1))
+    (fp_line (start -4.75 4.5) (end -4.75 -3.5) (layer F.Fab) (width 0.1))
+    (fp_line (start 4.75 4.5) (end -4.75 4.5) (layer F.Fab) (width 0.1))
+    (fp_text user %R (at 0 0 90) (layer F.Fab)
+      (effects (font (size 0.65 0.65) (thickness 0.125)))
+    )
+    (pad 20 smd rect (at -2.4 -4.75 270) (size 0.7 1.6) (layers F.Cu F.Paste F.Mask)
+      (net 108 "Net-(IC1-Pad20)"))
+    (pad 19 smd rect (at -1.2 -4.75 270) (size 0.7 1.6) (layers F.Cu F.Paste F.Mask)
+      (net 109 "Net-(IC1-Pad19)"))
+    (pad 18 smd rect (at 0 -4.75 270) (size 0.7 1.6) (layers F.Cu F.Paste F.Mask)
+      (net 119 "Net-(IC1-Pad18)"))
+    (pad 17 smd rect (at 1.2 -4.75 270) (size 0.7 1.6) (layers F.Cu F.Paste F.Mask)
+      (net 107 "Net-(IC1-Pad17)"))
+    (pad 16 smd rect (at 2.4 -4.75 270) (size 0.7 1.6) (layers F.Cu F.Paste F.Mask)
+      (net 106 "Net-(IC1-Pad16)"))
+    (pad 10 smd rect (at 2.4 4.75 270) (size 0.7 1.6) (layers F.Cu F.Paste F.Mask))
+    (pad 9 smd rect (at 1.2 4.75 270) (size 0.7 1.6) (layers F.Cu F.Paste F.Mask)
+      (net 1 GND))
+    (pad 8 smd rect (at 0 4.75 270) (size 0.7 1.6) (layers F.Cu F.Paste F.Mask)
+      (net 110 "Net-(BT1-Pad1)"))
+    (pad 7 smd rect (at -1.2 4.75 270) (size 0.7 1.6) (layers F.Cu F.Paste F.Mask)
+      (net 111 "Net-(C5-Pad1)"))
+    (pad 6 smd rect (at -2.4 4.75 270) (size 0.7 1.6) (layers F.Cu F.Paste F.Mask)
+      (net 1 GND))
+    (pad 15 smd rect (at 4.75 -2.4 270) (size 1.6 0.7) (layers F.Cu F.Paste F.Mask)
+      (net 118 "Net-(IC1-Pad15)"))
+    (pad 11 smd rect (at 4.75 2.4 270) (size 1.6 0.7) (layers F.Cu F.Paste F.Mask)
+      (net 117 "Net-(IC1-Pad11)"))
+    (pad 13 smd rect (at 4.75 0 270) (size 1.6 0.7) (layers F.Cu F.Paste F.Mask)
+      (net 104 "Net-(IC1-Pad13)"))
+    (pad 12 smd rect (at 4.75 1.2 270) (size 1.6 0.7) (layers F.Cu F.Paste F.Mask)
+      (net 103 "Net-(IC1-Pad12)"))
+    (pad 14 smd rect (at 4.75 -1.2 270) (size 1.6 0.7) (layers F.Cu F.Paste F.Mask)
+      (net 105 "Net-(IC1-Pad14)"))
+    (pad 5 smd rect (at -4.75 2.4 270) (size 1.6 0.7) (layers F.Cu F.Paste F.Mask)
+      (net 1 GND))
+    (pad 4 smd rect (at -4.75 1.2 270) (size 1.6 0.7) (layers F.Cu F.Paste F.Mask)
+      (net 1 GND))
+    (pad 3 smd rect (at -4.75 0 270) (size 1.6 0.7) (layers F.Cu F.Paste F.Mask)
+      (net 1 GND))
+    (pad 2 smd rect (at -4.75 -1.2 270) (size 1.6 0.7) (layers F.Cu F.Paste F.Mask)
+      (net 113 "Net-(IC1-Pad2)"))
+    (pad 1 smd rect (at -4.75 -2.4 270) (size 1.6 0.7) (layers F.Cu F.Paste F.Mask)
+      (net 1 GND))
+    (model ${KISYS3DMOD}/RF_GPS.3dshapes/Sierra_XM11X0.wrl
+      (at (xyz 0 0 0))
+      (scale (xyz 1 1 1))
+      (rotate (xyz 0 0 0))
+    )
   )
   (module Package_TO_SOT_THT:TO-220F-3_Vertical (layer F.Cu)
@@
       (at (xyz 0 0 0))
       (scale (xyz 1 1 1))
-      (rotate (xyz 0 0 0))
-    )
-  )
-  (module DashSight-PCB-Footprints:Sierra_XM11X0 (layer F.Cu)
-    (at 138.303 63.119 270)
-    (descr "QFN-20, Pitch 1.20 no EP, https://source.sierrawireless.com/resources/airprime/hardware_specs_user_guides/airprime_xm1100_product_technical_specification")
-    (tags "QFN-20 P1.20")
-    (attr smd)
-    (fp_text reference IC1 (at -3.1 -6.55 270) (layer F.SilkS)
-      (effects (font (size 1 1) (thickness 0.15)))
-    )
-    (fp_text value XM1110 (at 0 6.45 270) (layer F.Fab)
-      (effects (font (size 1 1) (thickness 0.15)))
-    )
-    (fp_line (start -4.6 -4.62) (end -3.6 -4.62) (layer F.SilkS) (width 0.12))
-    (fp_line (start 4.87 4.62) (end 4.87 3.62) (layer F.SilkS) (width 0.12))
-    (fp_line (start 3.87 4.62) (end 4.87 4.62) (layer F.SilkS) (width 0.12))
-    (fp_line (start -4.87 4.62) (end -4.87 3.62) (layer F.SilkS) (width 0.12))
-    (fp_line (start -3.87 4.62) (end -4.87 4.62) (layer F.SilkS) (width 0.12))
-    (fp_line (start 4.87 -4.62) (end 4.87 -3.62) (layer F.SilkS) (width 0.12))
-    (fp_line (start 3.87 -4.62) (end 4.87 -4.62) (layer F.SilkS) (width 0.12))
-    (fp_line (start 5.8 -5.8) (end -5.8 -5.8) (layer F.CrtYd) (width 0.05))
-    (fp_line (start 5.8 5.8) (end 5.8 -5.8) (layer F.CrtYd) (width 0.05))
-    (fp_line (start -5.8 5.8) (end 5.8 5.8) (layer F.CrtYd) (width 0.05))
-    (fp_line (start -5.8 -5.8) (end -5.8 5.8) (layer F.CrtYd) (width 0.05))
-    (fp_line (start 4.75 -4.5) (end 4.75 4.5) (layer F.Fab) (width 0.1))
-    (fp_line (start -3.75 -4.5) (end 4.75 -4.5) (layer F.Fab) (width 0.1))
-    (fp_line (start -4.75 -3.5) (end -3.75 -4.5) (layer F.Fab) (width 0.1))
-    (fp_line (start -4.75 4.5) (end -4.75 -3.5) (layer F.Fab) (width 0.1))
-    (fp_line (start 4.75 4.5) (end -4.75 4.5) (layer F.Fab) (width 0.1))
-    (fp_text user %R (at 0 0 270) (layer F.Fab)
-      (effects (font (size 0.65 0.65) (thickness 0.125)))
-    )
-    (pad 20 smd rect (at -2.4 -4.75 270) (size 0.7 1.6) (layers F.Cu F.Paste F.Mask)
-      (net 108 "Net-(IC1-Pad20)"))
-    (pad 19 smd rect (at -1.2 -4.75 270) (size 0.7 1.6) (layers F.Cu F.Paste F.Mask)
-      (net 109 "Net-(IC1-Pad19)"))
-    (pad 18 smd rect (at 0 -4.75 270) (size 0.7 1.6) (layers F.Cu F.Paste F.Mask)
-      (net 119 "Net-(IC1-Pad18)"))
-    (pad 17 smd rect (at 1.2 -4.75 270) (size 0.7 1.6) (layers F.Cu F.Paste F.Mask)
-      (net 107 "Net-(IC1-Pad17)"))
-    (pad 16 smd rect (at 2.4 -4.75 270) (size 0.7 1.6) (layers F.Cu F.Paste F.Mask)
-      (net 106 "Net-(IC1-Pad16)"))
-    (pad 10 smd rect (at 2.4 4.75 270) (size 0.7 1.6) (layers F.Cu F.Paste F.Mask))
-    (pad 9 smd rect (at 1.2 4.75 270) (size 0.7 1.6) (layers F.Cu F.Paste F.Mask)
-      (net 1 GND))
-    (pad 8 smd rect (at 0 4.75 270) (size 0.7 1.6) (layers F.Cu F.Paste F.Mask)
-      (net 110 "Net-(BT1-Pad1)"))
-    (pad 7 smd rect (at -1.2 4.75 270) (size 0.7 1.6) (layers F.Cu F.Paste F.Mask)
-      (net 111 "Net-(C5-Pad1)"))
-    (pad 6 smd rect (at -2.4 4.75 270) (size 0.7 1.6) (layers F.Cu F.Paste F.Mask)
-      (net 1 GND))
-    (pad 15 smd rect (at 4.75 -2.4 270) (size 1.6 0.7) (layers F.Cu F.Paste F.Mask)
-      (net 118 "Net-(IC1-Pad15)"))
-    (pad 11 smd rect (at 4.75 2.4 270) (size 1.6 0.7) (layers F.Cu F.Paste F.Mask)
-      (net 117 "Net-(IC1-Pad11)"))
-    (pad 13 smd rect (at 4.75 0 270) (size 1.6 0.7) (layers F.Cu F.Paste F.Mask)
-      (net 104 "Net-(IC1-Pad13)"))
-    (pad 12 smd rect (at 4.75 1.2 270) (size 1.6 0.7) (layers F.Cu F.Paste F.Mask)
-      (net 103 "Net-(IC1-Pad12)"))
-    (pad 14 smd rect (at 4.75 -1.2 270) (size 1.6 0.7) (layers F.Cu F.Paste F.Mask)
-      (net 105 "Net-(IC1-Pad14)"))
-    (pad 5 smd rect (at -4.75 2.4 270) (size 1.6 0.7) (layers F.Cu F.Paste F.Mask)
-      (net 1 GND))
-    (pad 4 smd rect (at -4.75 1.2 270) (size 1.6 0.7) (layers F.Cu F.Paste F.Mask)
-      (net 1 GND))
-    (pad 3 smd rect (at -4.75 0 270) (size 1.6 0.7) (layers F.Cu F.Paste F.Mask)
-      (net 1 GND))
-    (pad 2 smd rect (at -4.75 -1.2 270) (size 1.6 0.7) (layers F.Cu F.Paste F.Mask)
-      (net 113 "Net-(IC1-Pad2)"))
-    (pad 1 smd rect (at -4.75 -2.4 270) (size 1.6 0.7) (layers F.Cu F.Paste F.Mask)
-      (net 1 GND))
-    (model ${KISYS3DMOD}/RF_GPS.3dshapes/Sierra_XM11X0.wrl
-      (at (xyz 0 0 0))
-      (scale (xyz 1 1 1))

Commit message: pcb: Add my name to the PCB
Signed-off-by: Alistair Francis <alistair@alistair23.me>
Other:
- board text added: "Alistair Francis"
Changed lines of the file:
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@@
   (general
     (thickness 1.6)
-    (drawings 5)
+    (drawings 6)
     (tracks 539)
     (zones 0)
@@
     )
   )
-  (gr_text "DashSight v2.0-B" (at 183.388 55.372) (layer F.Cu)
+  (gr_text "Alistair Francis" (at 181.864 57.15) (layer F.Cu)
+    (effects (font (size 1.3 1.3) (thickness 0.3)))
+  )
+  (gr_text "DashSight v2.0-B" (at 183.388 54.864) (layer F.Cu)
     (effects (font (size 1.5 1.5) (thickness 0.3)))
   )
