File: DashSight-Mezzanine-Card.sch (KiCad schematic (older format))
At the start: 75 parts, among them IC2 ELM327, J1 Pi2 Connector, J2 Euler Connector, J3 Conn_Coaxial, J4 OBD2-DB9_Male, J5 Conn_02x05_Odd_Even, Q1 2N3904, Q2 2N3906, Q3 2N3906, Q4 2N3904, Q5 2N3904, Q6 2N3904, Q7 2N3904, SW1 SW_Push, SW2 SW_Push, U1 MCP2561-E/P, U2 LM317L_TO92, U3 LP2950-3.0_TO92, U4 ADuM1201AR, U5 NEO-M9N, Y1 4.0MHz

Commit message: sch: Update the microstrip numbers
Signed-off-by: Alistair Francis <alistair@alistair23.me>
Other:
- note added: "50 Ohm\nMicrostrip 0.2mm wide\nCopper Weight: 1oz/ft^2 \nLayer Thickness: 0.11mm\nSubstrate: FR4 TG130 (4.29)"
- note removed: "50 Ohm\nMicrostrip 1mm wide\nCopper Weight: 1oz/ft^2 \nBoard Thickness: 0.6mm\nSubstrate: FR4 TG130"
Changed lines of the file:
@@
 $EndComp
 Text Notes 3950 2700 0    60   ~ 0
-50 Ohm\nMicrostrip 1mm wide\nCopper Weight: 1oz/ft^2 \nBoard Thickness: 0.6mm\nSubstrate: FR4 TG130
+50 Ohm\nMicrostrip 0.2mm wide\nCopper Weight: 1oz/ft^2 \nLayer Thickness: 0.11mm\nSubstrate: FR4 TG130 (4.29)
 Connection ~ 4650 2750
 Connection ~ 3900 2750

Commit message: sch: Connect the PPS from GNSS
Signed-off-by: Alistair Francis <alistair@alistair23.me>
Connections:
- net labels added: I2C1_SCL, I2C1_SDA, PC7, PC8, PH9
- wire segments 249 -> 254
- no-connect marks 70 -> 64
Changed lines of the file:
@@
 NoConn ~ 15250 2850
 NoConn ~ 15250 2950
-NoConn ~ 15250 3350
 NoConn ~ 15250 3550
 NoConn ~ 15250 3650
@@
 NoConn ~ 14750 3650
 NoConn ~ 14750 3550
-NoConn ~ 14750 3450
-NoConn ~ 14750 3350
 NoConn ~ 14750 3150
-NoConn ~ 14750 3050
-NoConn ~ 14750 2950
 NoConn ~ 14700 5750
-NoConn ~ 14700 5850
-NoConn ~ 14700 5950
 NoConn ~ 14700 6050
 NoConn ~ 14700 6250
@@
 Wire Wire Line
 	3300 1350 2800 1350
-NoConn ~ 3500 3050
 NoConn ~ 2100 2750
 NoConn ~ 2100 2850
@@
 Wire Wire Line
 	4900 1500 4900 1600
+Text GLabel 15400 3350 2    60   Input ~ 0
+PC8
+Wire Wire Line
+	15250 3350 15400 3350
+NoConn ~ 14700 5950
+NoConn ~ 14700 5850
+Text GLabel 3500 3250 2    60   Output ~ 0
+PC8
+Text GLabel 14750 2950 0    60   BiDi ~ 0
+I2C1_SDA
+Text GLabel 14750 3050 0    60   Output ~ 0
+I2C1_SCL
+Text GLabel 14600 3350 0    60   Input ~ 0
+PC7
+Text GLabel 14600 3450 0    60   Input ~ 0
+PH9
+Wire Wire Line
+	14750 3350 14600 3350
+Wire Wire Line
+	14750 3450 14600 3450
+Wire Wire Line
+	3500 3050 3500 3250
+Wire Wire Line
+	3500 2750 4650 2750
 $EndSCHEMATC

Commit message: sch: Remove the Zener Diode from GNSS
Signed-off-by: Alistair Francis <alistair@alistair23.me>
Parts:
- removed D5: D_Zener, Diode_SMD:D_0201_0603Metric, symbol Device:D_Zener
Connections:
- wire segments 254 -> 249
Changed lines of the file:
@@
 	1750 3350 1750 3550
 Wire Wire Line
-	3900 3600 3900 3550
-Wire Wire Line
-	4650 3600 3900 3600
-Wire Wire Line
 	3650 3150 4250 3150
-Wire Wire Line
-	3900 3250 3900 2750
-Wire Wire Line
-	3500 2750 3900 2750
-$Comp
-L Device:D_Zener D5
-U 1 1 5E98F516
-P 3900 3400
-F 0 "D5" V 3854 3479 50  0000 L CNN
-F 1 "D_Zener" V 3945 3479 50  0000 L CNN
-F 2 "Diode_SMD:D_0201_0603Metric" H 3900 3400 50  0001 C CNN
-F 3 "DF2S5M4SL,L3F" H 3900 3400 50  0001 C CNN
-	1    3900 3400
-	0    1    1    0
-$EndComp
 Connection ~ 4650 3600
 Wire Wire Line
@@
 50 Ohm\nMicrostrip 0.2mm wide\nCopper Weight: 1oz/ft^2 \nLayer Thickness: 0.11mm\nSubstrate: FR4 TG130 (4.29)
 Connection ~ 4650 2750
-Connection ~ 3900 2750
-Wire Wire Line
-	3900 2750 4650 2750
 $Comp
 L Device:CP1 C5

Commit message: sch: Add the LSM9DS1 IMU
Signed-off-by: Alistair Francis <alistair@alistair23.me>
Parts:
- added C15, C16, C17: 0.1uF, Capacitor_SMD:C_0402_1005Metric, symbol Device:CP1
- added C18: 10uF, Capacitor_THT:CP_Radial_D4.0mm_P1.50mm, symbol Device:CP1
- added C9: 10nF (16V), Capacitor_SMD:C_0402_1005Metric, symbol Device:CP1
- added R31, R32, R33, R34, R35, R36: 10K, Resistors_SMD:R_0603, symbol Device:R
- added R37, R38: 2.2K, Resistors_SMD:R_0603, symbol Device:R
- added U6: LSM9DS1, Package_LGA:LGA-24L_3x3.5mm_P0.43mm, symbol Sensor_Motion:LSM9DS1
Connections:
- wire segments 249 -> 303
- no-connect marks 64 -> 67

Commit message: sch: Fixup resistor types
Signed-off-by: Alistair Francis <alistair@alistair23.me>
Parts:
- R12, R31, R32, R33, R34, R35, R36, R37, R38: footprint Resistors_SMD:R_0603 -> Resistor_SMD:R_0603_1608Metric
Changed lines of the file:
@@
 F 0 "R12" V 9080 5250 50  0000 C CNN
 F 1 "10K" V 9000 5250 50  0000 C CNN
-F 2 "Resistors_SMD:R_0603" V 8930 5250 50  0001 C CNN
+F 2 "Resistor_SMD:R_0603_1608Metric" V 8930 5250 50  0001 C CNN
 F 3 "RC0603FR-0710KL" H 9000 5250 50  0001 C CNN
 	1    9000 5250
@@
 F 0 "R32" V 1280 8800 50  0000 C CNN
 F 1 "10K" V 1200 8800 50  0000 C CNN
-F 2 "Resistors_SMD:R_0603" V 1130 8800 50  0001 C CNN
+F 2 "Resistor_SMD:R_0603_1608Metric" V 1130 8800 50  0001 C CNN
 F 3 "RC0603FR-0710KL" H 1200 8800 50  0001 C CNN
 	1    1200 8800
@@
 F 0 "R35" V 3730 8550 50  0000 C CNN
 F 1 "10K" V 3650 8550 50  0000 C CNN
-F 2 "Resistors_SMD:R_0603" V 3580 8550 50  0001 C CNN
+F 2 "Resistor_SMD:R_0603_1608Metric" V 3580 8550 50  0001 C CNN
 F 3 "RC0603FR-0710KL" H 3650 8550 50  0001 C CNN
 	1    3650 8550
@@
 F 0 "R36" V 4180 8600 50  0000 C CNN
 F 1 "10K" V 4100 8600 50  0000 C CNN
-F 2 "Resistors_SMD:R_0603" V 4030 8600 50  0001 C CNN
+F 2 "Resistor_SMD:R_0603_1608Metric" V 4030 8600 50  0001 C CNN
 F 3 "RC0603FR-0710KL" H 4100 8600 50  0001 C CNN
 	1    4100 8600
@@
 F 0 "R31" V 1080 8900 50  0000 C CNN
 F 1 "10K" V 1000 8900 50  0000 C CNN
-F 2 "Resistors_SMD:R_0603" V 930 8900 50  0001 C CNN
+F 2 "Resistor_SMD:R_0603_1608Metric" V 930 8900 50  0001 C CNN
 F 3 "RC0603FR-0710KL" H 1000 8900 50  0001 C CNN
 	1    1000 8900
@@
 F 0 "R34" V 2180 8300 50  0000 C CNN
 F 1 "10K" V 2100 8300 50  0000 C CNN
-F 2 "Resistors_SMD:R_0603" V 2030 8300 50  0001 C CNN
+F 2 "Resistor_SMD:R_0603_1608Metric" V 2030 8300 50  0001 C CNN
 F 3 "RC0603FR-0710KL" H 2100 8300 50  0001 C CNN
 	1    2100 8300
@@
 F 0 "R33" V 1980 8400 50  0000 C CNN
 F 1 "10K" V 1900 8400 50  0000 C CNN
-F 2 "Resistors_SMD:R_0603" V 1830 8400 50  0001 C CNN
+F 2 "Resistor_SMD:R_0603_1608Metric" V 1830 8400 50  0001 C CNN
 F 3 "RC0603FR-0710KL" H 1900 8400 50  0001 C CNN
 	1    1900 8400
@@
 F 0 "R38" V 14180 2800 50  0000 C CNN
 F 1 "2.2K" V 14100 2800 50  0000 C CNN
-F 2 "Resistors_SMD:R_0603" V 14030 2800 50  0001 C CNN
-F 3 "" H 14100 2800 50  0001 C CNN
+F 2 "Resistor_SMD:R_0603_1608Metric" V 14030 2800 50  0001 C CNN
+F 3 "RC0603FR-072K2L" H 14100 2800 50  0001 C CNN
 	1    14100 2800
 	1    0    0    -1
@@
 F 0 "R37" V 13980 2900 50  0000 C CNN
 F 1 "2.2K" V 13900 2900 50  0000 C CNN
-F 2 "Resistors_SMD:R_0603" V 13830 2900 50  0001 C CNN
-F 3 "" H 13900 2900 50  0001 C CNN
+F 2 "Resistor_SMD:R_0603_1608Metric" V 13830 2900 50  0001 C CNN
+F 3 "RC0603FR-072K2L" H 13900 2900 50  0001 C CNN
 	1    13900 2900
 	1    0    0    -1

Commit message: sch: Improve the GNSS breakout headers
Signed-off-by: Alistair Francis <alistair@alistair23.me>
Parts:
- removed H1: Safeboot, Connector_PinHeader_2.54mm:PinHeader_1x01_P2.54mm_Vertical, symbol Mechanical:MountingHole_Pad
- removed H2: Reset, Connector_PinHeader_2.54mm:PinHeader_1x01_P2.54mm_Vertical, symbol Mechanical:MountingHole_Pad
- added J6: Safeboot, Connector_PinHeader_2.54mm:PinHeader_1x01_P2.54mm_Vertical, symbol Connector_Generic:Conn_01x01
- added J7: Reset, Connector_PinHeader_2.54mm:PinHeader_1x01_P2.54mm_Vertical, symbol Connector_Generic:Conn_01x01
Changed lines of the file:
@@
 	2700 1600 3950 1600
 NoConn ~ 2100 3050
-$Comp
-L Mechanical:MountingHole_Pad H1
-U 1 1 5EE6A9A7
-P 1400 2950
-F 0 "H1" H 1500 2999 50  0000 L CNN
-F 1 "Safeboot" H 1500 2908 50  0000 L CNN
-F 2 "Connector_PinHeader_2.54mm:PinHeader_1x01_P2.54mm_Vertical" H 1400 2950 50  0001 C CNN
-F 3 "" H 1400 2950 50  0001 C CNN
-	1    1400 2950
-	1    0    0    -1
-$EndComp
-$Comp
-L Mechanical:MountingHole_Pad H2
-U 1 1 5EE6E3F9
-P 1750 3650
-F 0 "H2" H 1650 3607 50  0000 R CNN
-F 1 "Reset" H 1650 3698 50  0000 R CNN
-F 2 "Connector_PinHeader_2.54mm:PinHeader_1x01_P2.54mm_Vertical" H 1750 3650 50  0001 C CNN
-F 3 "" H 1750 3650 50  0001 C CNN
-	1    1750 3650
-	-1   0    0    1
-$EndComp
 Wire Wire Line
 	1400 3050 1400 3250
@@
 	13900 3050 14750 3050
 Connection ~ 13900 3050
+$Comp
+L Connector_Generic:Conn_01x01 J7
+U 1 1 5F1BAEC9
+P 1750 3750
+F 0 "J7" V 1622 3830 50  0000 L CNN
+F 1 "Reset" V 1713 3830 50  0000 L CNN
+F 2 "Connector_PinHeader_2.54mm:PinHeader_1x01_P2.54mm_Vertical" H 1750 3750 50  0001 C CNN
+F 3 "" H 1750 3750 50  0001 C CNN
+	1    1750 3750
+	0    1    1    0
+$EndComp
+$Comp
+L Connector_Generic:Conn_01x01 J6
+U 1 1 5F1BDA69
+P 1400 2850
+F 0 "J6" V 1364 2762 50  0000 R CNN
+F 1 "Safeboot" V 1273 2762 50  0000 R CNN
+F 2 "Connector_PinHeader_2.54mm:PinHeader_1x01_P2.54mm_Vertical" H 1400 2850 50  0001 C CNN
+F 3 "" H 1400 2850 50  0001 C CNN
+	1    1400 2850
+	0    -1   -1   0
+$EndComp
 $EndSCHEMATC

Commit message: sch: Update the schematic to include Qwiic
Signed-off-by: Alistair Francis <alistair@alistair23.me>
Parts:
- added J10, J11, J12, J13, J8, J9: QWIIC_CONNECTORJS-1MM, DashSight:qwiic_connector, symbol sparkfun:QWIIC_CONNECTORJS-1MM
Connections:
- wire segments 303 -> 315
Other:
- note added: "ELM327 OBDII"
- note added: "I2C Expansion Qwiic Connectors"
- note added: "Inertial Measurement Unit (IMU)"
- moved on the sheet: C15, C16, C17, C18, C9, R31, R32, R33, R34, R35, R36

Commit message: sch: Update the headers and power supply
Signed-off-by: Alistair Francis <alistair@alistair23.me>
Parts:
- J6, J7: footprint Connector_PinHeader_2.54mm:PinHeader_1x01_P2.54mm_Vertical -> Connector_PinHeader_1.00mm:PinHeader_1x01_P1.00mm_Vertical
Connections:
- wire segments 315 -> 321
- no-connect marks 67 -> 64
Changed lines of the file:
@@
 NoConn ~ 14750 3850
 NoConn ~ 14750 3750
-NoConn ~ 14750 3650
 NoConn ~ 14750 3550
 NoConn ~ 14750 3150
-NoConn ~ 14700 5750
 NoConn ~ 14700 6050
 NoConn ~ 14700 6250
 NoConn ~ 14700 6350
 NoConn ~ 14700 6450
-NoConn ~ 14700 6550
 NoConn ~ 14700 6650
 NoConn ~ 14700 6750
@@
 F 0 "J7" V 1622 3830 50  0000 L CNN
 F 1 "Reset" V 1713 3830 50  0000 L CNN
-F 2 "Connector_PinHeader_2.54mm:PinHeader_1x01_P2.54mm_Vertical" H 1750 3750 50  0001 C CNN
+F 2 "Connector_PinHeader_1.00mm:PinHeader_1x01_P1.00mm_Vertical" H 1750 3750 50  0001 C CNN
 F 3 "" H 1750 3750 50  0001 C CNN
 	1    1750 3750
@@
 F 0 "J6" V 1364 2762 50  0000 R CNN
 F 1 "Safeboot" V 1273 2762 50  0000 R CNN
-F 2 "Connector_PinHeader_2.54mm:PinHeader_1x01_P2.54mm_Vertical" H 1400 2850 50  0001 C CNN
+F 2 "Connector_PinHeader_1.00mm:PinHeader_1x01_P1.00mm_Vertical" H 1400 2850 50  0001 C CNN
 F 3 "" H 1400 2850 50  0001 C CNN
 	1    1400 2850
@@
 Text Notes 2450 4650 0    60   ~ 0
 I2C Expansion Qwiic Connectors
+$Comp
+L power:+3.3V #PWR?
+U 1 1 5EB35FB4
+P 14200 3550
+F 0 "#PWR?" H 14200 3400 50  0001 C CNN
+F 1 "+3.3V" H 14215 3723 50  0000 C CNN
+F 2 "" H 14200 3550 50  0001 C CNN
+F 3 "" H 14200 3550 50  0001 C CNN
+	1    14200 3550
+	1    0    0    -1
+$EndComp
+Wire Wire Line
+	14750 3650 14200 3650
+Wire Wire Line
+	14200 3650 14200 3550
+$Comp
+L power:+3.3V #PWR?
+U 1 1 5EB7237F
+P 14450 5600
+F 0 "#PWR?" H 14450 5450 50  0001 C CNN
+F 1 "+3.3V" H 14465 5773 50  0000 C CNN
+F 2 "" H 14450 5600 50  0001 C CNN
+F 3 "" H 14450 5600 50  0001 C CNN
+	1    14450 5600
+	1    0    0    -1
+$EndComp
+Wire Wire Line
+	14700 5750 14450 5750
+Wire Wire Line
+	14450 5750 14450 5600
+Wire Wire Line
+	14700 6550 14450 6550
+Wire Wire Line
+	14450 6550 14450 5750
+Connection ~ 14450 5750
 $EndSCHEMATC
