File: DashSight-Mezzanine-Card.sch (KiCad schematic (older format))
At the start: 94 parts, among them IC2 ELM327, J1 Pi2 Connector, J10 QWIIC_CONNECTORJS-1MM, J11 QWIIC_CONNECTORJS-1MM, J12 QWIIC_CONNECTORJS-1MM, J13 QWIIC_CONNECTORJS-1MM, J2 Euler Connector, J3 Conn_Coaxial, J4 OBD2-DB9_Male, J5 Conn_02x05_Odd_Even, J6 Safeboot, J7 Reset, J8 QWIIC_CONNECTORJS-1MM, J9 QWIIC_CONNECTORJS-1MM, Q1 2N3904, Q2 2N3906, Q3 2N3906, Q4 2N3904, Q5 2N3904, Q6 2N3904, Q7 2N3904, SW1 SW_Push, SW2 SW_Push, U1 MCP2561-E/P, U2 LM317L_TO92, U3 LP2950-3.0_TO92, U4 ADuM1201AR, U5 NEO-M9N, U6 LSM9DS1, Y1 4.0MHz

Commit message: Breakout some GPIOs and fixup remaining issues
Signed-off-by: Alistair Francis <alistair@alistair23.me>
Parts:
- added J14: 1W-PC16, Connector_PinHeader_1.27mm:PinHeader_1x03_P1.27mm_Vertical, symbol Connector_Generic:Conn_01x03
- added J15: 1W-PC9, Connector_PinHeader_1.27mm:PinHeader_1x03_P1.27mm_Vertical, symbol Connector_Generic:Conn_01x03
Connections:
- net labels added: PC16, PC9
- wire segments 321 -> 327
- no-connect marks 64 -> 62
Other:
- note added: "1-Wire GPIO Connections"
Changed lines of the file:
@@
 NoConn ~ 15250 4650
 NoConn ~ 15250 4750
-NoConn ~ 14750 4650
-NoConn ~ 14750 4550
 NoConn ~ 14750 4450
 NoConn ~ 14750 4350
@@
 I2C Expansion Qwiic Connectors
 $Comp
-L power:+3.3V #PWR?
+L power:+3.3V #PWR069
 U 1 1 5EB35FB4
 P 14200 3550
-F 0 "#PWR?" H 14200 3400 50  0001 C CNN
+F 0 "#PWR069" H 14200 3400 50  0001 C CNN
 F 1 "+3.3V" H 14215 3723 50  0000 C CNN
 F 2 "" H 14200 3550 50  0001 C CNN
@@
 	14200 3650 14200 3550
 $Comp
-L power:+3.3V #PWR?
+L power:+3.3V #PWR070
 U 1 1 5EB7237F
 P 14450 5600
-F 0 "#PWR?" H 14450 5450 50  0001 C CNN
+F 0 "#PWR070" H 14450 5450 50  0001 C CNN
 F 1 "+3.3V" H 14465 5773 50  0000 C CNN
 F 2 "" H 14450 5600 50  0001 C CNN
@@
 	14450 6550 14450 5750
 Connection ~ 14450 5750
+$Comp
+L Connector_Generic:Conn_01x03 J14
+U 1 1 5ED3A7C7
+P 8600 2650
+F 0 "J14" H 8518 2325 50  0000 C CNN
+F 1 "1W-PC16" H 8518 2416 50  0000 C CNN
+F 2 "Connector_PinHeader_1.27mm:PinHeader_1x03_P1.27mm_Vertical" H 8600 2650 50  0001 C CNN
+F 3 "" H 8600 2650 50  0001 C CNN
+	1    8600 2650
+	-1   0    0    1
+$EndComp
+Text GLabel 8800 2650 2    60   Output ~ 0
+PC16
+Text GLabel 14600 4650 0    60   BiDi ~ 0
+PC16
+Text GLabel 14600 4550 0    60   BiDi ~ 0
+PC9
+$Comp
+L power:GND #PWR065
+U 1 1 5ED3EFCB
+P 8800 2750
+F 0 "#PWR065" H 8800 2500 50  0001 C CNN
+F 1 "GND" H 8805 2577 50  0000 C CNN
+F 2 "" H 8800 2750 50  0001 C CNN
+F 3 "" H 8800 2750 50  0001 C CNN
+	1    8800 2750
+	1    0    0    -1
+$EndComp
+$Comp
+L power:+3V3 #PWR066
+U 1 1 5ED402EF
+P 8950 2500
+F 0 "#PWR066" H 8950 2350 50  0001 C CNN
+F 1 "+3V3" H 8965 2673 50  0000 C CNN
+F 2 "" H 8950 2500 50  0001 C CNN
+F 3 "" H 8950 2500 50  0001 C CNN
+	1    8950 2500
+	1    0    0    -1
+$EndComp
+Wire Wire Line
+	8800 2550 8950 2550
+Wire Wire Line
+	8950 2550 8950 2500
+$Comp
+L Connector_Generic:Conn_01x03 J15
+U 1 1 5ED62042
+P 9550 2650
+F 0 "J15" H 9468 2325 50  0000 C CNN
+F 1 "1W-PC9" H 9468 2416 50  0000 C CNN
+F 2 "Connector_PinHeader_1.27mm:PinHeader_1x03_P1.27mm_Vertical" H 9550 2650 50  0001 C CNN
+F 3 "" H 9550 2650 50  0001 C CNN
+	1    9550 2650
+	-1   0    0    1
+$EndComp
+Text GLabel 9750 2650 2    60   Output ~ 0
+PC9
+$Comp
+L power:GND #PWR067
+U 1 1 5ED62049
+P 9750 2750
+F 0 "#PWR067" H 9750 2500 50  0001 C CNN
+F 1 "GND" H 9755 2577 50  0000 C CNN
+F 2 "" H 9750 2750 50  0001 C CNN
+F 3 "" H 9750 2750 50  0001 C CNN
+	1    9750 2750
+	1    0    0    -1
+$EndComp
+$Comp
+L power:+3V3 #PWR068
+U 1 1 5ED6204F
+P 9900 2500
+F 0 "#PWR068" H 9900 2350 50  0001 C CNN
+F 1 "+3V3" H 9915 2673 50  0000 C CNN
+F 2 "" H 9900 2500 50  0001 C CNN
+F 3 "" H 9900 2500 50  0001 C CNN
+	1    9900 2500
+	1    0    0    -1
+$EndComp
+Wire Wire Line
+	9750 2550 9900 2550
+Wire Wire Line
+	9900 2550 9900 2500
+Text Notes 8700 2150 0    60   ~ 0
+1-Wire GPIO Connections
+Wire Wire Line
+	14750 4550 14600 4550
+Wire Wire Line
+	14600 4650 14750 4650
 $EndSCHEMATC

Commit message: Only support 6 Qwiic connections
I was worried I couuldn't fit the cables in with 6

Signed-off-by: Alistair Francis <alistair@alistair23.me>
Parts:
- removed J11, J12, J13: QWIIC_CONNECTORJS-1MM, DashSight:qwiic_connector, symbol sparkfun:QWIIC_CONNECTORJS-1MM
Connections:
- wire segments 327 -> 321
Other:
- moved on the sheet: C15, C16, C17, C18, C9, R31, R32, R33, R34, R35, R36

Commit message: sch: Update some of the footprints
Signed-off-by: Alistair Francis <alistair@alistair23.me>
Parts:
- J1: footprint Pin_Headers:Pin_Header_Straight_2x20_Pitch2.54mm -> Connector_PinSocket_2.54mm:PinSocket_2x20_P2.54mm_Vertical
- J2: footprint Pin_Headers:Pin_Header_Straight_2x17_Pitch2.54mm -> Connector_PinSocket_2.54mm:PinSocket_2x17_P2.54mm_Vertical
- J3: footprint Connectors:SMA_THT_Jack_Straight -> Connector_Coaxial:SMA_Amphenol_132134_Vertical
- J5: footprint Connector_PinHeader_2.54mm:PinHeader_2x05_P2.54mm_Vertical -> Connector_PinSocket_2.54mm:PinSocket_2x05_P2.54mm_Vertical
- JP1, JP2: footprint Pin_Headers:Pin_Header_Straight_1x02_Pitch2.54mm -> Connector_PinHeader_2.54mm:PinHeader_1x02_P2.54mm_Vertical
- U1: footprint Housings_DIP:DIP-8_W7.62mm -> Package_DIP:DIP-8_W7.62mm
- U2: footprint TO_SOT_Packages_THT:TO-92_Inline_Narrow_Oval -> Package_TO_SOT_THT:TO-92_Inline
- U4: footprint Housings_SOIC:SOIC-8_3.9x4.9mm_Pitch1.27mm -> Package_SO:SOIC-8_3.9x4.9mm_P1.27mm
- Y1: footprint Crystals:Crystal_HC49-U_Vertical -> Crystal:Crystal_HC49-U_Vertical
Changed lines of the file:
@@
 F 0 "Y1" H 9100 6550 50  0000 C CNN
 F 1 "4.0MHz" H 9100 6250 50  0000 C CNN
-F 2 "Crystals:Crystal_HC49-U_Vertical" H 9100 6400 50  0001 C CNN
+F 2 "Crystal:Crystal_HC49-U_Vertical" H 9100 6400 50  0001 C CNN
 F 3 "ECS-040-20-4X-DU " H 9100 6400 50  0001 C CNN
 	1    9100 6400
@@
 F 0 "U1" H 11050 4000 50  0000 L CNN
 F 1 "MCP2561-E/P" H 11550 4000 50  0000 L CNN
-F 2 "Housings_DIP:DIP-8_W7.62mm" H 11450 3150 50  0001 C CIN
+F 2 "Package_DIP:DIP-8_W7.62mm" H 11450 3150 50  0001 C CIN
 F 3 "MCP2561-E/P" H 11450 3650 50  0001 C CNN
 	1    11450 3650
@@
 F 0 "U2" H 8250 7325 50  0000 C CNN
 F 1 "LM317L_TO92" H 8400 7325 50  0000 L CNN
-F 2 "TO_SOT_Packages_THT:TO-92_Inline_Narrow_Oval" H 8400 7425 50  0001 C CIN
+F 2 "Package_TO_SOT_THT:TO-92_Inline" H 8400 7425 50  0001 C CIN
 F 3 "LM317LZX" H 8400 7200 50  0001 C CNN
 	1    8400 7200
@@
 F 0 "J1" H 15000 4867 50  0000 C CNN
 F 1 "Pi2 Connector" H 15000 4776 50  0000 C CNN
-F 2 "Pin_Headers:Pin_Header_Straight_2x20_Pitch2.54mm" H 14950 3750 50  0001 C CNN
+F 2 "Connector_PinSocket_2.54mm:PinSocket_2x20_P2.54mm_Vertical" H 14950 3750 50  0001 C CNN
 F 3 "PPPC202LFBN-RC" H 14950 3750 50  0001 C CNN
 	1    14950 3750
@@
 F 0 "J2" H 14950 7567 50  0000 C CNN
 F 1 "Euler Connector" H 14950 7476 50  0000 C CNN
-F 2 "Pin_Headers:Pin_Header_Straight_2x17_Pitch2.54mm" H 14900 6550 50  0001 C CNN
+F 2 "Connector_PinSocket_2.54mm:PinSocket_2x17_P2.54mm_Vertical" H 14900 6550 50  0001 C CNN
 F 3 "PPPC172LFBN-RC" H 14900 6550 50  0001 C CNN
 	1    14900 6550
@@
 F 0 "U4" H 12950 7017 50  0000 C CNN
 F 1 "ADuM1201AR" H 12950 6926 50  0000 C CNN
-F 2 "Housings_SOIC:SOIC-8_3.9x4.9mm_Pitch1.27mm" H 12950 6150 50  0001 C CIN
+F 2 "Package_SO:SOIC-8_3.9x4.9mm_P1.27mm" H 12950 6150 50  0001 C CIN
 F 3 "ADuM1201AR" H 12950 6450 50  0001 C CNN
 	1    12950 6550
@@
 F 0 "JP2" H 11700 1714 50  0000 C CNN
 F 1 "Vbat-JP" H 11700 1623 50  0000 C CNN
-F 2 "Pin_Headers:Pin_Header_Straight_1x02_Pitch2.54mm" H 11700 1450 50  0001 C CNN
+F 2 "Connector_PinHeader_2.54mm:PinHeader_1x02_P2.54mm_Vertical" H 11700 1450 50  0001 C CNN
 F 3 "61300211121" H 11700 1450 50  0001 C CNN
 	1    11700 1450
@@
 F 0 "JP1" H 9900 1514 50  0000 C CNN
 F 1 "DCIn-JP" H 9900 1423 50  0000 C CNN
-F 2 "Pin_Headers:Pin_Header_Straight_1x02_Pitch2.54mm" H 9900 1250 50  0001 C CNN
+F 2 "Connector_PinHeader_2.54mm:PinHeader_1x02_P2.54mm_Vertical" H 9900 1250 50  0001 C CNN
 F 3 "61300211121" H 9900 1250 50  0001 C CNN
 	1    9900 1250
@@
 F 0 "J5" H 14950 8917 50  0000 C CNN
 F 1 "Conn_02x05_Odd_Even" H 14950 8826 50  0000 C CNN
-F 2 "Connector_PinHeader_2.54mm:PinHeader_2x05_P2.54mm_Vertical" H 14900 8500 50  0001 C CNN
+F 2 "Connector_PinSocket_2.54mm:PinSocket_2x05_P2.54mm_Vertical" H 14900 8500 50  0001 C CNN
 F 3 "PPPC052LFBN-RC" H 14900 8500 50  0001 C CNN
 	1    14900 8500
@@
 F 0 "J3" H 5349 2726 50  0000 L CNN
 F 1 "Conn_Coaxial" H 5349 2635 50  0000 L CNN
-F 2 "Connectors:SMA_THT_Jack_Straight" H 5250 2750 50  0001 C CNN
+F 2 "Connector_Coaxial:SMA_Amphenol_132134_Vertical" H 5250 2750 50  0001 C CNN
 F 3 "CONREVSMA002-G" H 5250 2750 50  0001 C CNN
 	1    5250 2750

Commit message: sch: Add a jumper to enable SPI for the IMU
Signed-off-by: Alistair Francis <alistair@alistair23.me>
Parts:
- added JP3, JP4, JP5, JP6, JP7, JP8: Jumper, Jumper:SolderJumper-2_P1.3mm_Bridged_Pad1.0x1.5mm, symbol Device:Jumper
Connections:
- net labels added: PC15, PH7, SPI0_CLK, SPI0_MISO, SPI0_MOSI, SPI_SEL_CLK, SPI_SEL_CS1, SPI_SEL_CS2, SPI_SEL_SDA, SPI_SEL_SDOAG, SPI_SEL_SDOM
- wire segments 321 -> 329
- no-connect marks 62 -> 57
Other:
- moved on the sheet: R32

Commit message: Revert "sch: Add a jumper to enable SPI for the IMU"
This reverts commit a1cdc124bf6f11fea9068c468dfdf75d15ab77d8.

Signed-off-by: Alistair Francis <alistair@alistair23.me>
Parts:
- removed JP3, JP4, JP5, JP6, JP7, JP8: Jumper, Jumper:SolderJumper-2_P1.3mm_Bridged_Pad1.0x1.5mm, symbol Device:Jumper
Connections:
- net labels removed: PC15, PH7, SPI0_CLK, SPI0_MISO, SPI0_MOSI, SPI_SEL_CLK, SPI_SEL_CS1, SPI_SEL_CS2, SPI_SEL_SDA, SPI_SEL_SDOAG, SPI_SEL_SDOM
- wire segments 329 -> 321
- no-connect marks 57 -> 62
Other:
- moved on the sheet: R32

Commit message: Update based on BOM avaliability
Signed-off-by: Alistair Francis <alistair@alistair23.me>
Parts:
- D4: footprint Resistors_SMD:R_0402 -> Diode_SMD:D_0603_1608Metric
Changed lines of the file:
@@
 F 0 "D4" V 4496 1071 50  0000 R CNN
 F 1 "0.5A/40V/420mV" V 4405 1071 50  0000 R CNN
-F 2 "Resistors_SMD:R_0402" H 4450 1150 50  0001 C CNN
-F 3 "VSKY05401006-G4-08" H 4450 1150 50  0001 C CNN
+F 2 "Diode_SMD:D_0603_1608Metric" H 4450 1150 50  0001 C CNN
+F 3 "CDBVRL140-HF" H 4450 1150 50  0001 C CNN
 	1    4450 1150
 	0    -1   -1   0

Commit message: Revert "Revert "sch: Add a jumper to enable SPI for the IMU""
This reverts commit c516a7607144a3527f6f3ebaa38245544a61c706.

Signed-off-by: Alistair Francis <alistair@alistair23.me>
Parts:
- added JP3, JP4, JP5, JP6, JP7, JP8: Jumper, Jumper:SolderJumper-2_P1.3mm_Bridged_Pad1.0x1.5mm, symbol Device:Jumper
Connections:
- net labels added: PC15, PH7, SPI0_CLK, SPI0_MISO, SPI0_MOSI, SPI_SEL_CLK, SPI_SEL_CS1, SPI_SEL_CS2, SPI_SEL_SDA, SPI_SEL_SDOAG, SPI_SEL_SDOM
- wire segments 321 -> 329
- no-connect marks 62 -> 57
Other:
- moved on the sheet: R32

Commit message: sch: Update all of the pin connections
Signed-off-by: Alistair Francis <alistair@alistair23.me>
Parts:
- removed J15: 1W-PC9, Connector_PinHeader_1.27mm:PinHeader_1x03_P1.27mm_Vertical, symbol Connector_Generic:Conn_01x03
- removed JP3, JP4, JP5, JP6, JP7, JP8: Jumper, Jumper:SolderJumper-2_P1.3mm_Bridged_Pad1.0x1.5mm, symbol Device:Jumper
- removed R31, R32, R33, R34, R35, R36: 10K, Resistor_SMD:R_0603_1608Metric, symbol Device:R
Connections:
- net labels added: PC11, PC4, PH5, PH6
- net labels removed: PC15, PC16, PC8, PC9, PH9, SPI_SEL_CLK, SPI_SEL_CS1, SPI_SEL_CS2, SPI_SEL_SDA, SPI_SEL_SDOAG, SPI_SEL_SDOM
- wire segments 329 -> 311
- no-connect marks 57 -> 58
